Commit message: fix(description): give the camera housing collision geometry
`camera_body` declared visual geometry and an inertia but no `<collision>`
element, so MoveIt did not see the camera housing as an obstacle and a future C3
approach could be accepted that clips it. The housing was visible in RViz and
invisible to planning, which is the failure mode that looks correct until a
trajectory is executed.

- add a `<collision>` box to `camera_body` and drive both the visual and the
  collision box from one `camera_body_size` property, so the two cannot drift
  into two independent literals
- keep the `0.05 0.05 0.03` dimensions, no origin on either element, and leave
  `camera_post`, `camera_optical` and all three camera joints untouched
- add tests/unit/test_robot_description_camera_collision.py, which expands the
  description with xacro and fails closed when the collision element is removed,
  when the two boxes diverge, when an origin offsets one from the other, or when
  the tree grows a second root or a duplicate link
- document that `camera_optical` is a convention frame and must stay
  collision-free while `camera_body` is the solid housing

Collision geometry here is a planning obstacle only. It is not continuous
collision safety and does not authorize trajectory execution.

Closes #261.

Task Packet: docs/task_packets/description-261-camera-body-collision.json
Gate: make lint, make test, make contract, make scenario-check, make
      golden-check, make context-check

Also reformats hardware/mechanical/tools/generate_artifacts.py, which `ruff
format --check` flagged on main after the #328 change. Cosmetic only.

File: robot/description/workbench.urdf.xacro (robot description, xacro)
@@ -169,9 +169,16 @@
             rpy="0 0 0"/>
   </joint>
+  <!-- The camera housing is an obstacle for planning, so it carries collision
+       geometry with the same box as its visual. A visual-only body is invisible
+       to MoveIt, which then accepts approaches that clip the housing. -->
+  <xacro:property name="camera_body_size" value="0.05 0.05 0.03"/>
   <link name="camera_body">
     <visual>
-      <geometry><box size="0.05 0.05 0.03"/></geometry>
+      <geometry><box size="${camera_body_size}"/></geometry>
       <material name="black"/>
     </visual>
+    <collision>
+      <geometry><box size="${camera_body_size}"/></geometry>
+    </collision>
     <xacro:box_inertia m="0.1" x="0.05" y="0.05" z="0.03"/>
   </link>
